File: Hardware/ESP32_Thing_Plus_UFL.brd (EAGLE design)
At the start: 22.9 x 58.4 mm, 107 parts, among them Q1 2.5A/30V, Q2 MBT3904DW1T1, U1 MCP73831, U2 ESP-WROOM-32NARROW, U3 AP2112K-3.3V, U4 CP210X

Commit message: switched to u.fl module and modified the CP2104 VBUS input
-u.fl module swapped out
-added standoffs and new measures
-moved product name and logo to top of board
-added in voltage split circuit to vbus input to CP2104
-connected VREGIN pin on CP2104 to 3.3V (previously was connected to vbus)
-changed value of R1 to 2.2K
-added C2 and C3 for additional decoupling caps near CP2104
Parts:
- removed U$58: (no value), buzzard_labels (42):ESP32_THING_PLUS0
- removed U2: ESP-WROOM-32NARROW, SparkFun-RF:ESP-WROOM-32-NARROW
- added C2: 0.1uF, SparkFun-Capacitors:0402-TIGHT
- added C3: 4.7uF, SparkFun-Capacitors:0402-TIGHT
- added H3, H4: STAND-OFFTIGHT, SparkFun-Hardware:STAND-OFF-TIGHT
- added LOGO5: SFE_LOGO_NAME_FLAME.1_INCH, SparkFun-Aesthetics:SFE_LOGO_NAME_FLAME_.1
- added R9: 33k, SparkFun-Resistors:0402-TIGHT
- added U$24: (no value), output:ESP32_THING_PLUS0
- added U5: ESP-WROOM-3232U-NARROW, esp-wroom-32u:ESP-WROOM-32U-NARROW
- R1: value 1k -> 2.2K; device SparkFun-Resistors:0603 -> SparkFun-Resistors:0402
- R5: value 10 -> 22k; device SparkFun-Resistors:0603 -> SparkFun-Resistors:0402-TIGHT
- moved LOGO3 5.66 mm to (11.4, 54.5)
- moved FD1 4.32 mm to (17.7, 57.7)
- moved FD2 4.32 mm to (17.7, 57.7)
- moved R5 2.29 mm to (18.2, 16.9)
Connections:
- removed net 20: U2.32
- removed net N$3: R5.2, U4.7, U4.8
- new net N$4: R5.1, R9.2, U4.8
- net 0: now also U5.25; no longer U2.25
- net 12: now also U5.14; no longer U2.14
- net 13: now also U5.16; no longer U2.16
- net 14: now also U5.13; no longer U2.13
- net 15: now also U5.23; no longer U2.23
- net 16: now also U5.27; no longer U2.27
- net 17: now also U5.28; no longer U2.28
- net 21: now also U5.33; no longer U2.33
- net 27: now also U5.12; no longer U2.12
- net 3.3V: now also C2.1, C3.1, U4.7, U5.2; no longer U2.2
- net 32: now also U5.8; no longer U2.8
- net 33: now also U5.9; no longer U2.9
- net A0: now also U5.11; no longer U2.11
- net A1: now also U5.10; no longer U2.10
- net A2: now also U5.6; no longer U2.6
- net A3: now also U5.5; no longer U2.5
- net A4: now also U5.4; no longer U2.4
- net A5: now also U5.26; no longer U2.26
- net CHIP_PU: now also U5.3; no longer U2.3
- net GND: now also C2.2, C3.2, R9.1, U5.1, U5.15, U5.38, U5.GND; no longer U2.1, U2.15, U2.38, U2.GND
- net MISO: now also U5.31; no longer U2.31
- net MOSI: now also U5.30; no longer U2.30
- net RX: now also U5.35; no longer U2.35
- net SCK: now also U5.29; no longer U2.29
- net SCL: now also U5.36; no longer U2.36
- net SDA: now also U5.37; no longer U2.37
- net TX: now also U5.34; no longer U2.34
- net V_USB: now also R5.2; no longer R5.1
Routing:
- net N$4: track 0.00 -> 9.85 mm
- net 3.3V: track 24.0 -> 31.0 mm
- net N$3: track 6.89 -> 0.00 mm
- net GND: track 38.5 -> 41.6 mm, vias 18 -> 19
Other:
- board text added: "Revised by: Pete Lewis (u.fl)"
- board text added: "v10"
- board text removed: "Units in inches"
- board text removed: "v20"

Commit message: post design review changes
-changed R1 to a 10K (pullup on RSTB on CP2102)
-nudged U1 (and nearby passives) down to make more space around pin 13 LED.
-changed all 0402 "standard" footprints to use the "tight". re-routed as necessary.
-made all 4.7uF caps the same 0402 part
-made all 1.0uF caps (qty 2) the same 0402 part (X5R)
Parts:
- C10: device SparkFun-Capacitors:0402 -> SparkFun-Capacitors:0402-TIGHT
- C19, C6, C7: device SparkFun-Capacitors:0603 -> SparkFun-Capacitors:0402-TIGHT
- R1: value 2.2K -> 10k; device SparkFun-Resistors:0402 -> SparkFun-Resistors:0603
- R8: value 100K -> 100k; device SparkFun-Resistors:0402 -> SparkFun-Resistors:0402-TIGHT
- moved U1 0.89 mm to (6.35, 24.5)
- moved R3 0.63 mm to (18.9, 10.2)
- moved R6 0.63 mm to (4.57, 27.6)
- moved C10 0.38 mm to (9.53, 28.2)
- moved C6 0.38 mm to (3.81, 24.9)
- moved D3 0.38 mm to (6.10, 29.2)
- moved R2 0.38 mm to (18.9, 13.7)
- moved U$53 0.38 mm to (2.79, 29.2)
Routing:
- net GND: track 41.6 -> 45.2 mm
- net 3.3V: track 31.0 -> 34.0 mm
- net N$4: track 9.85 -> 12.4 mm
- net VIN: track 12.7 -> 13.9 mm
- net V_USB: track 13.6 -> 14.5 mm
- net N$17: track 9.74 -> 9.11 mm

Commit message: new buzzards, swapped out Miso/Mosi naming
Parts:
- removed U$1: (no value), buzzard_labels (37):#RESET0
- removed U$13: (no value), buzzard_labels (37):A03
- removed U$14: (no value), buzzard_labels (37):A14
- removed U$15: (no value), buzzard_labels (37):A25
- removed U$16: (no value), buzzard_labels (37):A36
- removed U$17: (no value), buzzard_labels (37):A47
- removed U$18: (no value), buzzard_labels (37):A58
- removed U$2: (no value), buzzard_labels (37):3V31
- removed U$20: (no value), buzzard_labels (37):GND2
- removed U$47: (no value), buzzard_labels (39):SCK20
- removed U$48: (no value), buzzard_labels (4):GND21
- removed U$49: (no value), buzzard_labels (4):NC22
- removed U$50: (no value), buzzard_labels (39):VUSB8
- removed U$51: (no value), buzzard_labels (39):EN9
- removed U$52: (no value), buzzard_labels (39):VBAT10
- removed U$53: (no value), buzzard_labels (39):137
- removed U$54: (no value), buzzard_labels (40):MISO0
- removed U$55: (no value), buzzard_labels (40):MOSI1
- removed U$56: (no value), buzzard_labels (41):CHG1
- removed U$57: (no value), buzzard_labels (41):RESET0
- removed U$6: (no value), buzzard_labels (7):16#RX11
- removed U$60: (no value), buzzard_labels (4):3V323
- removed U$61: (no value), buzzard_labels (4):RST24
- removed U$62: (no value), buzzard_labels:00
- removed U$63: (no value), buzzard_labels (5):5#SCK2
- removed U$64: (no value), buzzard_labels:NC0
- removed U$65: (no value), buzzard_labels:ESP32_THING_PLUS0
- removed U$66: (no value), buzzard_labels (5):18#MOSI1
- removed U$67: (no value), buzzard_labels (5):19#MISO0
- removed U$7: (no value), buzzard_labels (7):17#TX10
- removed U$9: (no value), buzzard_labels (8):210
- added LOGO6: QWIIC_LOGO_5MM, SparkFun-Aesthetics:QWIIC_5MM
- added U$25: (no value), output:SDA0
- added U$26: (no value), output:SCL0
- added U$58: (no value), output:140
- added U$68: (no value), output:320
- added U$69: (no value), output:150
- added U$70: (no value), output:330
- added U$71: (no value), output:270
- added U$72: (no value), output:120
- added U$73, U$74: (no value), output:130
- added U$75: (no value), output:VUSB0
- added U$76: (no value), output:EN0
- added U$77: (no value), output:VBAT0
- added U$78: (no value), output:CHG0
- added U$79: (no value), output:RESET0
- added U$80: (no value), output:RST0
- added U$81: (no value), output:3V30
- added U$82: (no value), output:NC0
- added U$83: (no value), output:GND0
- added U$84: (no value), output:A00
- added U$85: (no value), output:A10
- added U$86: (no value), output:A20
- added U$87: (no value), output:A30
- added U$88: (no value), output:A40
- added U$89: (no value), output:A50
- added U$90: (no value), output:SCK0
- added U$93: (no value), output:160
- added U$94: (no value), output:170
- added U$95: (no value), output:210
- added U$96: (no value), output:00
- U$10: device buzzard_labels (37):2721 -> output:#18#COPI#0
- U$11: device buzzard_labels (37):3218 -> output:#5#SCK#0
- U$12: device buzzard_labels (37):3320 -> output:#A5#0
- U$19: device buzzard_labels (37):EN26 -> output:#A4#0
- U$21: device buzzard_labels (14):22#SCL1 -> output:#A3#0
- U$22: device buzzard_labels (14):23#SDA0 -> output:#A2#0
- U$23: device buzzard_labels (37):QWIIC27 -> output:DI0
- U$27: device buzzard_labels (37):VBAT25 -> output:#A1#0
- U$28: device buzzard_labels (37):VUSB24 -> output:#A0#0
- U$29: device buzzard_labels (4):SDA1 -> output:DO0
- U$3: device buzzard_labels (37):1323 -> output:#21#0
- U$30: device buzzard_labels (4):SCL0 -> output:ESP_THING_PLUS_0
- U$31: device buzzard_labels (4):142 -> output:#23#SDA#0
- U$32: device buzzard_labels (4):323 -> output:#GND#0
- U$33: device buzzard_labels (4):154 -> output:#22#SCL#0
- U$34: device buzzard_labels (4):335 -> output:#14#0
- U$35: device buzzard_labels (4):276 -> output:#32#0
- U$36: device buzzard_labels (4):127 -> output:#15#0
- U$37: device buzzard_labels (4):138 -> output:#33#0
- U$38: device buzzard_labels (4):219 -> output:#27#0
- U$39: device buzzard_labels (4):1710 -> output:#12#0
- U$4: device buzzard_labels (37):1417 -> output:#17#TX1#0
- U$40: device buzzard_labels (4):1611 -> output:#13#0
- U$41: device buzzard_labels (4):A515 -> output:#VUSB#0
- U$42: device buzzard_labels (4):A416 -> output:#VBAT#0
- U$43: device buzzard_labels (4):A317 -> output:#EN#0
- U$44: device buzzard_labels (4):A218 -> output:#NC#0
- U$45: device buzzard_labels (4):A119 -> output:#3V3#0
- U$46: device buzzard_labels (4):A020 -> output:##RESET##0
- U$5: device buzzard_labels (37):1519 -> output:#16#RX1#0
- U$8: device buzzard_labels (8):121 -> output:#19#CIPO#0
- moved U$23 34.8 mm to (21.6, 43.2), turned to 0 degrees
- moved U$32 30.2 mm to (21.1, 21.6), flipped to the bottom
- moved U$3 26.0 mm to (21.1, 52.1)
- moved U$22 25.9 mm to (21.1, 29.2)
- moved U$29 24.3 mm to (21.6, 40.6)
- moved U$39 23.2 mm to (1.78, 34.3), flipped to the bottom
- moved U$40 23.2 mm to (1.78, 31.8), flipped to the bottom
- moved U$38 23.1 mm to (1.78, 36.8), flipped to the bottom
- moved U$21 21.7 mm to (21.1, 31.8)
- moved U$42 20.3 mm to (1.78, 24.1), flipped to the bottom
- moved U$41 19.5 mm to (1.78, 29.2), flipped to the bottom
- moved U$8 19.1 mm to (21.1, 44.5)
- moved U$43 18.7 mm to (1.78, 26.7), flipped to the bottom
- moved U$30 18.6 mm to (11.5, 33.9), flipped to the bottom, turned to 270 degrees
- moved U$19 17.4 mm to (21.1, 34.3)
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Connections:
- net MISO renamed CIPO
- net MOSI renamed COPI

Commit message: aesthetic changes from post review review
-Change CIPO and COPI pin names in symbol to SDI/SDO
-Updated product name bottom silk to include "32"
-Removed extra top silk flame logo at bottom right (since we had room for the full name and flame logo at the top.
-changed silk names for DI/DO to SDI/SDO for more consitency in schematic/board naming.
Parts:
- removed LOGO1: SFE_LOGO_FLAME.1_INCH, SparkFun-Aesthetics:SFE_LOGO_FLAME_.1
- removed U$23: (no value), output:DI0
- removed U$29: (no value), output:DO0
- removed U$30: (no value), output:ESP_THING_PLUS_0
- added U$1: (no value), output:ESP32_THING_PLUS_0
- added U$2: (no value), output:SDI0
- added U$6: (no value), output:SDO0
- moved LOGO2 15.3 mm to (20.8, 6.10)
Changed lines of the file:
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@@
 <drawing>
 <settings>
-<setting alwaysvectorfont="yes"/>
+<setting alwaysvectorfont="no"/>
 <setting keepoldvectorfont="yes"/>
 <setting verticaltext="up"/>
@@
 <layers>
 <layer number="1" name="Top" color="4" fill="1" visible="yes" active="yes"/>
-<layer number="2" name="Route2" color="1" fill="3" visible="yes" active="yes"/>
-<layer number="15" name="Route15" color="4" fill="6" visible="yes" active="yes"/>
+<layer number="2" name="Route2" color="1" fill="3" visible="no" active="yes"/>
+<layer number="15" name="Route15" color="4" fill="6" visible="no" active="yes"/>
 <layer number="16" name="Bottom" color="1" fill="1" visible="yes" active="yes"/>
 <layer number="17" name="Pads" color="2" fill="1" visible="yes" active="yes"/>
@@
 <attribute name="VALUE" x="16.51" y="31.369" size="0.6096" layer="27" font="vector" ratio="20" rot="R180" align="top-center"/>
 </element>
-<element name="LOGO2" library="SparkFun-Aesthetics" package="OSHW-LOGO-MINI" value="OSHW-LOGOMINI" x="5.588" y="4.826" smashed="yes"/>
+<element name="LOGO2" library="SparkFun-Aesthetics" package="OSHW-LOGO-MINI" value="OSHW-LOGOMINI" x="20.828" y="6.096" smashed="yes"/>
 <element name="J3" library="SparkFun-Connectors" package="1X04_1MM_RA" value="" x="5.08" y="9.398" smashed="yes" rot="R270">
 <attribute name="NAME" x="2.921" y="10.795" size="0.6096" layer="25" font="vector" ratio="20" rot="R270"/>
@@
 <attribute name="VALUE" value="100k" x="9.271" y="21.336" size="0.6096" layer="27" font="vector" ratio="20" align="top-center"/>
 </element>
-<element name="LOGO1" library="SparkFun-Aesthetics" package="SFE_LOGO_FLAME_.1" value="SFE_LOGO_FLAME.1_INCH" x="18.669" y="5.461" smashed="yes"/>
 <element name="LOGO3" library="SparkFun-Aesthetics" package="SFE_LOGO_NAME_FLAME_.1" value="SFE_LOGO_NAME_FLAME.1_INCH" x="11.43" y="54.483" smashed="yes" rot="MR0"/>
 <element name="LOGO4" library="SparkFun-Aesthetics" package="FOUR_LAYER_WARNING" value="FOUR_LAYER_WARNING" x="30.48" y="39.37" smashed="yes"/>
@@
 <element name="U$96" library="output" package="00" value="" x="9.5504" y="14.1478" smashed="yes"/>
 <element name="LOGO6" library="SparkFun-Aesthetics" package="QWIIC_5MM" value="QWIIC_LOGO_5MM" x="6.858" y="9.525" smashed="yes" rot="R270"/>
-<element name="U$23" library="output" package="DI0" value="" x="21.59" y="43.18" smashed="yes"/>
-<element name="U$29" library="output" package="DO0" value="" x="21.59" y="40.64" smashed="yes"/>
-<element name="U$30" library="output" package="ESP_THING_PLUS_0" value="" x="11.4554" y="33.909" smashed="yes" rot="MR270"/>
 <element name="U$31" library="output" package="#23#SDA#0" value="" x="1.778" y="52.07" smashed="yes" rot="MR0"/>
 <element name="U$33" library="output" package="#22#SCL#0" value="" x="1.778" y="49.53" smashed="yes" rot="MR0"/>
@@
 <element name="U$45" library="output" package="#3V3#0" value="" x="21.082" y="16.51" smashed="yes" rot="MR0"/>
 <element name="U$46" library="output" package="##RESET##0" value="" x="21.082" y="13.97" smashed="yes" rot="MR0"/>
+<element name="U$1" library="output" package="ESP32_THING_PLUS_0" value="" x="11.43" y="33.02" smashed="yes" rot="MR270"/>
+<element name="U$2" library="output" package="SDI0" value="" x="21.6154" y="43.18" smashed="yes"/>
+<element name="U$6" library="output" package="SDO0" value="" x="21.6916" y="40.64" smashed="yes"/>
 </elements>
 <signals>

Commit message: Run of checklist catches
-vector font in sch
-flag label on NET "0"
-changes top silk on RST pin to include active low marking
Parts:
- removed U$80: (no value), output:RST0
- added U$7: (no value), output:#RST#0
Changed lines of the file:
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@@
 <element name="U$78" library="output" package="CHG0" value="" x="16.51" y="5.715" smashed="yes" rot="R90"/>
 <element name="U$79" library="output" package="RESET0" value="" x="16.1036" y="14.1986" smashed="yes"/>
-<element name="U$80" library="output" package="RST0" value="" x="21.59" y="12.7" smashed="yes"/>
 <element name="U$81" library="output" package="3V30" value="" x="21.59" y="15.24" smashed="yes"/>
 <element name="U$82" library="output" package="NC0" value="" x="21.59" y="17.78" smashed="yes"/>
@@
 <element name="U$2" library="output" package="SDI0" value="" x="21.6154" y="43.18" smashed="yes"/>
 <element name="U$6" library="output" package="SDO0" value="" x="21.6916" y="40.64" smashed="yes"/>
+<element name="U$7" library="output" package="#RST#0" value="" x="21.5392" y="12.4714" smashed="yes"/>
 </elements>
 <signals>

Commit message: changing library part names/descriptions to the 32EU
Parts:
- U5: value ESP-WROOM-3232U-NARROW -> ESP-WROOM-32EU; device esp-wroom-32u:ESP-WROOM-32U-NARROW -> esp-wroom-32u:ESP-WROOM-32EU-NARROW
Changed lines of the file:
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@@
 <attribute name="VALUE" x="20.32" y="0.889" size="0.6096" layer="27" font="vector" ratio="20" align="top-center"/>
 </element>
-<element name="U5" library="esp-wroom-32u" package="ESP-WROOM-32U-NARROW" value="ESP-WROOM-3232U-NARROW" x="11.43" y="44.45" smashed="yes" rot="R90">
+<element name="U5" library="esp-wroom-32u" package="ESP-WROOM-32EU-NARROW" value="ESP-WROOM-32EU" x="11.43" y="44.45" smashed="yes" rot="R90">
 <attribute name="NAME" x="5.855" y="43.307" size="0.8128" layer="25" rot="R270" align="center"/>
 <attribute name="PROD_ID" value="IC-15442" x="11.43" y="44.45" size="1.778" layer="27" rot="R90" display="off"/>
