File: Hardware/ESP32_Thing_Plus_UFL.brd (EAGLE design)
At the start: 22.9 x 58.4 mm, 112 parts, among them Q1 2.5A/30V, Q2 MBT3904DW1T1, U1 MCP73831, U3 AP2112K-3.3V, U4 CP210X, U5 ESP-WROOM-32EU

Commit message: Silk Update
Updated silk on bottom
Added "Doot" to GPIO0 button
Parts:
- removed LOGO3: SFE_LOGO_NAME_FLAME.1_INCH, SparkFun-Aesthetics:SFE_LOGO_NAME_FLAME_.1
- U$1: device output:ESP32_THING_PLUS_0 -> output:DOOT0
- moved U$1 19.3 mm to (10.2, 13.7), flipped to the top, turned to 0 degrees
- moved U$96 7.11 mm to (9.47, 7.04)
- moved U$79 0.48 mm to (16.1, 13.7)
- renumbered LOGO5 to LOGO1
Routing:
- net GND: track 45.5 -> 46.3 mm
